Commit message: urdf_config8 works

File: src/urdf_v4/urdf/urdf_v4.urdf (robot description, URDF)
Before this commit: robot urdf_v4, 11 links, 10 joints
Links:
- removed link gripper_arm1
- removed link gripper_arm2
- removed link gripper_link_gear1
- removed link gripper_link_gear2
- added link leg1, mass 0.0106754375169454; collision mesh filename=package://urdf_v16/meshes/leg1.STL; visual mesh filename=package://urdf_v16/meshes/leg1.STL
- added link leg2, mass 0.0106754461770056; collision mesh filename=package://urdf_v16/meshes/leg2.STL; visual mesh filename=package://urdf_v16/meshes/leg2.STL
- added link servo_gear1, mass 0.00438273139903777; collision mesh filename=package://urdf_v16/meshes/servo_gear1.STL; visual mesh filename=package://urdf_v16/meshes/servo_gear1.STL
- added link servo_gear2, mass 0.00438273139817732; collision mesh filename=package://urdf_v16/meshes/servo_gear2.STL; visual mesh filename=package://urdf_v16/meshes/servo_gear2.STL
- link gripper_base: mass 0.066955061265398 -> 0.0669550622960312; geometry collision mesh filename=package://urdf_v16/meshes/gripper_base.STL; visual mesh filename=package://urdf_v16/meshes/gripper_base.STL
Joints:
- removed joint joint_10
- removed joint joint_9
- added joint jleg1: type fixed, parent servo_gear1, child leg1, origin xyz=-0.019057 -0.019896 0.0073322 rpy=1.5563 0.0046149 -0.0046825, axis 0.99999 0 -0.0046829
- added joint jleg2: type fixed, parent servo_gear2, child leg2, origin xyz=0.0091903 -0.019693 0.021245 rpy=1.5563 0.0046149 -0.0046825, axis 0 0 0
- joint joint_5: origin xyz=0 0 0.098960745637557 rpy=0 0 0 -> xyz=0 0 0.098961 rpy=0 0 0
- joint joint_6: origin xyz=0.00101787720548718 0.0025808298232558 -0.67198995308091 rpy=0 0 0 -> xyz=0.00098171 -0.000501 -0.66696 rpy=0 0 0
- joint joint_7: axis 0.99989 -0.013774 -0.0046829 -> 0.99999 0 -0.0046829; child gripper_link_gear1 -> servo_gear1; origin xyz=0.0022853 -0.016581 0.73698 rpy=0 0 0.013775 -> xyz=0.0093777 -0.013452 0.73231 rpy=-1.5563 0.0046149 0.0046825
- joint joint_8: axis -0.99989 0.013774 0.0046829 -> 0.99999 0 -0.0046829; child gripper_link_gear2 -> servo_gear2; mimic joint=joint_7 multiplier=-1 offset=0 -> joint=joint_7 multiplier=1 offset=0; origin xyz=0.0022853 0.011419 0.73698 rpy=-1.5621 -0.0047239 -3.1369 -> xyz=-0.00062209 0.014501 0.73236 rpy=-1.5563 -0.0047509 -3.1369
